Commit message: new urdf added this time

File: sr_ronex_arm_description/robots/sr_ronex_arm.urdf (robot description, URDF)
Before this commit: robot sr_ronex_arm_description, 8 links, 7 joints
Joints:
- removed joint tooth_j1
- removed joint tooth_j2
- added joint gripper: type prismatic, parent link_5, child tooth_1, origin xyz=0 0 0.021 rpy=0 0 0, axis 0 -1 0, limit lower=0 upper=0.016 effort=0 velocity=0.05
- added joint gripper_2: type prismatic, parent link_5, child tooth_2, origin xyz=0 0 0.021 rpy=0 0 0, axis 0 1 0, limit lower=0 upper=0.016 effort=0 velocity=0.05, mimic joint=gripper multiplier=1 offset=0

Commit message: 1st three joints working

File: sr_ronex_arm_description/robots/sr_ronex_arm.urdf (robot description, URDF)
Before this commit: robot sr_ronex_arm_description, 8 links, 7 joints
Joints:
- joint joint_1: limit lower=-2.3 upper=2.3 effort=0 velocity=3 -> lower=-2.3 upper=2.3 effort=100 velocity=3
- joint joint_2: limit lower=-1.57 upper=2.36 effort=0 velocity=3 -> lower=-1.57 upper=2.36 effort=100.0 velocity=3
- joint joint_3: limit lower=-2.4 upper=2.4 effort=0 velocity=3 -> lower=-2.4 upper=2.4 effort=100 velocity=3

Commit message: joints all working

File: sr_ronex_arm_description/robots/sr_ronex_arm.urdf (robot description, URDF)
Before this commit: robot sr_ronex_arm_description, 8 links, 7 joints
Joints:
- joint gripper: limit lower=0 upper=0.016 effort=0 velocity=0.05 -> lower=0 upper=0.016 effort=100 velocity=0.05
- joint gripper_2: limit lower=0 upper=0.016 effort=0 velocity=0.05 -> lower=0 upper=0.016 effort=100 velocity=0.05
- joint joint_4: limit lower=-1.5 upper=1.5 effort=0 velocity=3 -> lower=-1.5 upper=1.5 effort=100 velocity=3
- joint joint_5: limit lower=-1.5 upper=1.5 effort=0 velocity=3 -> lower=-1.5 upper=1.5 effort=100 velocity=3

Commit message: Got hybrid control on j1

File: sr_ronex_arm_description/robots/sr_ronex_arm.urdf (robot description, URDF)
Before this commit: robot sr_ronex_arm_description, 8 links, 7 joints
Joints:
- joint joint_1: limit lower=-2.3 upper=2.3 effort=100 velocity=3 -> lower=-2.3 upper=2.3 effort=100 velocity=.9

Commit message: improved

File: sr_ronex_arm_description/robots/sr_ronex_arm.urdf (robot description, URDF)
Before this commit: robot sr_ronex_arm_description, 8 links, 7 joints
Joints:
- joint joint_2: limit lower=-1.57 upper=2.36 effort=100.0 velocity=3 -> lower=-1.5 upper=1.5 effort=100.0 velocity=.5

Commit message: improved v control

File: sr_ronex_arm_description/robots/sr_ronex_arm.urdf (robot description, URDF)
Before this commit: robot sr_ronex_arm_description, 8 links, 7 joints
Joints:
- joint joint_1: limit lower=-2.3 upper=2.3 effort=100 velocity=.9 -> lower=-2.3 upper=2.3 effort=100 velocity=2

Commit message: Working p/control

File: sr_ronex_arm_description/robots/sr_ronex_arm.urdf (robot description, URDF)
Before this commit: robot sr_ronex_arm_description, 8 links, 7 joints
Joints:
- joint joint_2: limit lower=-1.5 upper=1.5 effort=100.0 velocity=.5 -> lower=-1.5 upper=1.5 effort=100.0 velocity=1
- joint joint_3: limit lower=-2.4 upper=2.4 effort=100 velocity=3 -> lower=-2.4 upper=2.4 effort=100 velocity=1

Commit message: script

File: sr_ronex_arm_description/robots/sr_ronex_arm.urdf (robot description, URDF)
Before this commit: robot sr_ronex_arm_description, 8 links, 7 joints
Joints:
- joint joint_1: limit lower=-2.3 upper=2.3 effort=100 velocity=2 -> lower=-2.3 upper=2.3 effort=100 velocity=1
- joint joint_2: limit lower=-1.5 upper=1.5 effort=100.0 velocity=1 -> lower=-1 upper=1.85 effort=100.0 velocity=1
- joint joint_4: limit lower=-1.5 upper=1.5 effort=100 velocity=3 -> lower=-1.5 upper=1.5 effort=100 velocity=1
- joint joint_5: limit lower=-1.5 upper=1.5 effort=100 velocity=3 -> lower=-1.5 upper=1.5 effort=100 velocity=1
